Commit message: add rviz

File: src/arm_description/urdf/Arm.urdf (robot description, URDF)
Before this commit: robot Arm, 46 links, 45 joints
Links:
- link EE_link: geometry collision mesh filename=package://arm_description/meshes/EE_link.STL; visual mesh filename=package://arm_description/meshes/EE_link.STL
- link EE_sensor1_camera_link: geometry collision mesh filename=package://arm_description/meshes/EE_sensor1_camera_link.STL; visual mesh filename=package://arm_description/meshes/EE_sensor1_camera_link.STL
- link EE_sensor1_link: geometry collision mesh filename=package://arm_description/meshes/EE_sensor1_link.STL; visual mesh filename=package://arm_description/meshes/EE_sensor1_link.STL
- link EE_sensor1_tof_link: geometry collision mesh filename=package://arm_description/meshes/EE_sensor1_tof_link.STL; visual mesh filename=package://arm_description/meshes/EE_sensor1_tof_link.STL
- link EE_sensor2_camera_link: geometry collision mesh filename=package://arm_description/meshes/EE_sensor2_camera_link.STL; visual mesh filename=package://arm_description/meshes/EE_sensor2_camera_link.STL
- link EE_sensor2_link: geometry collision mesh filename=package://arm_description/meshes/EE_sensor2_link.STL; visual mesh filename=package://arm_description/meshes/EE_sensor2_link.STL
- link EE_sensor2_tof_link: geometry collision mesh filename=package://arm_description/meshes/EE_sensor2_tof_link.STL; visual mesh filename=package://arm_description/meshes/EE_sensor2_tof_link.STL
- link base_link: geometry collision mesh filename=package://arm_description/meshes/base_link.STL; visual mesh filename=package://arm_description/meshes/base_link.STL
- link link1: geometry collision mesh filename=package://arm_description/meshes/link1.STL; visual mesh filename=package://arm_description/meshes/link1.STL
- link link2: geometry collision mesh filename=package://arm_description/meshes/link2.STL; visual mesh filename=package://arm_description/meshes/link2.STL
- link link2_sensor1_camera_link: geometry collision mesh filename=package://arm_description/meshes/link2_sensor1_camera_link.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; visual mesh filename=package://arm_description/meshes/link2_sensor1_camera_link.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
- link link2_sensor1_link: geometry collision mesh filename=package://arm_description/meshes/link2_sensor1_link.STL; visual mesh filename=package://arm_description/meshes/link2_sensor1_link.STL
- link link2_sensor1_tof_link: geometry collision mesh filename=package://arm_description/meshes/link2_sensor1_tof_link.STL; visual mesh filename=package://arm_description/meshes/link2_sensor1_tof_link.STL
- link link2_sensor2_camera_link: geometry collision mesh filename=package://arm_description/meshes/link2_sensor2_camera_link.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; visual mesh filename=package://arm_description/meshes/link2_sensor2_camera_link.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
- link link2_sensor2_link: geometry collision mesh filename=package://arm_description/meshes/link2_sensor2_link.STL; visual mesh filename=package://arm_description/meshes/link2_sensor2_link.STL
- link link2_sensor2_tof_link: geometry collision mesh filename=package://arm_description/meshes/link2_sensor2_tof_link.STL; visual mesh filename=package://arm_description/meshes/link2_sensor2_tof_link.STL
- link link3: geometry collision mesh filename=package://arm_description/meshes/link3.STL; visual mesh filename=package://arm_description/meshes/link3.STL
- link link3_sensor1_camera_link: geometry collision mesh filename=package://arm_description/meshes/link3_sensor1_camera_link.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; visual mesh filename=package://arm_description/meshes/link3_sensor1_camera_link.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
- link link3_sensor1_link: geometry collision mesh filename=package://arm_description/meshes/link3_sensor1_link.STL; visual mesh filename=package://arm_description/meshes/link3_sensor1_link.STL
- link link3_sensor1_tof_link: geometry collision mesh filename=package://arm_description/meshes/link3_sensor1_tof_link.STL; visual mesh filename=package://arm_description/meshes/link3_sensor1_tof_link.STL
- link link3_sensor2_camera_link: geometry collision mesh filename=package://arm_description/meshes/link3_sensor2_camera_link.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; visual mesh filename=package://arm_description/meshes/link3_sensor2_camera_link.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
- link link3_sensor2_link: geometry collision mesh filename=package://arm_description/meshes/link3_sensor2_link.STL; visual mesh filename=package://arm_description/meshes/link3_sensor2_link.STL
- link link3_sensor2_tof_link: geometry collision mesh filename=package://arm_description/meshes/link3_sensor2_tof_link.STL; visual mesh filename=package://arm_description/meshes/link3_sensor2_tof_link.STL
- link link4: geometry collision mesh filename=package://arm_description/meshes/link4.STL; visual mesh filename=package://arm_description/meshes/link4.STL
- link link4_sensor1_camera_link: geometry collision mesh filename=package://arm_description/meshes/link4_sensor1_camera_link.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; visual mesh filename=package://arm_description/meshes/link4_sensor1_camera_link.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
- link link4_sensor1_link: geometry collision mesh filename=package://arm_description/meshes/link4_sensor1_link.STL; visual mesh filename=package://arm_description/meshes/link4_sensor1_link.STL
- link link4_sensor1_tof_link: geometry collision mesh filename=package://arm_description/meshes/link4_sensor1_tof_link.STL; visual mesh filename=package://arm_description/meshes/link4_sensor1_tof_link.STL
- link link4_sensor2_camera_link: geometry collision mesh filename=package://arm_description/meshes/link4_sensor2_camera_link.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; visual mesh filename=package://arm_description/meshes/link4_sensor2_camera_link.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
- link link4_sensor2_link: geometry collision mesh filename=package://arm_description/meshes/link4_sensor2_link.STL; visual mesh filename=package://arm_description/meshes/link4_sensor2_link.STL
- link link4_sensor2_tof_link: geometry collision mesh filename=package://arm_description/meshes/link4_sensor2_tof_link.STL; visual mesh filename=package://arm_description/meshes/link4_sensor2_tof_link.STL
- link wrist_link1: geometry collision mesh filename=package://arm_description/meshes/wrist_link1.STL; visual mesh filename=package://arm_description/meshes/wrist_link1.STL
- link wrist_link2: geometry collision mesh filename=package://arm_description/meshes/wrist_link2.STL; visual mesh filename=package://arm_description/meshes/wrist_link2.STL
- link wrist_link3: geometry collision mesh filename=package://arm_description/meshes/wrist_link3.STL; visual mesh filename=package://arm_description/meshes/wrist_link3.STL

Commit message: velocity execution baseline and add EE interactive marker target

File: src/arm_description/urdf/Arm.urdf (robot description, URDF)
Before this commit: robot Arm, 46 links, 45 joints
Links:
- link EE_sensor1_link: mass 0.0280853097776282 -> 0.028085
- link base_link: mass 0.766851050223606 -> 1.8984
- link link1: mass 2.22318567608356 -> 3.7184
- link link2: mass 1.25469347638256 -> 1.2547
- link link3: mass 0.582589401925533 -> 1.5556
- link link4: mass 0.499691951248306 -> 1.8227
- link wrist_link1: mass 0.165249310681186 -> 0.51524
- link wrist_link2: mass 0.113563263335891 -> 0.46355
- link wrist_link3: mass 0.0627633465287199 -> 0.062763
Joints:
- joint joint1: limit lower=-3.14 upper=3.14 effort=100 velocity=100 -> lower=-3.14 upper=3.14 effort=170 velocity=20.106193
- joint joint2: limit lower=-2.3 upper=2.3 effort=100 velocity=100 -> lower=-2.3 upper=2.3 effort=300 velocity=11.100294
- joint joint3: limit lower=-3.14 upper=3.14 effort=100 velocity=100 -> lower=-3.14 upper=3.14 effort=148 velocity=11.728613
- joint joint4: limit lower=-2.65 upper=2.65 effort=100 velocity=100 -> lower=-2.65 upper=2.65 effort=148 velocity=11.728613
- joint wrist_joint1: limit lower=-3.14 upper=3.14 effort=100 velocity=100 -> lower=-3.14 upper=3.14 effort=30 velocity=9.215338
- joint wrist_joint2: limit lower=-3.14 upper=3.14 effort=100 velocity=100 -> lower=-3.14 upper=3.14 effort=30 velocity=9.215338
- joint wrist_joint3: limit lower=-1.2 upper=1.2 effort=100 velocity=100 -> lower=-1.2 upper=1.2 effort=30 velocity=9.215338
