Commit message: Phase E1: add EE ToF sensors to Gazebo

File: src/arm_description/urdf/Arm.urdf (robot description, URDF)
Before this commit: robot Arm, 46 links, 45 joints
Links:
- added link EE_sensor1_tof_gz_link, mass 0.000001
- added link EE_sensor2_tof_gz_link, mass 0.000001
Joints:
- added joint EE_sensor1_tof_gz_joint: type fixed, parent EE_sensor1_tof_link, child EE_sensor1_tof_gz_link, origin xyz=0 0 0 rpy=1.5707963267949 -1.5707963267949 0, axis 0 0 0
- added joint EE_sensor2_tof_gz_joint: type fixed, parent EE_sensor2_tof_link, child EE_sensor2_tof_gz_link, origin xyz=0 0 0 rpy=1.5707963267949 -1.5707963267949 0, axis 0 0 0
