Commit message: Fix link2 self-filter collision geometry

File: src/arm_description/urdf/Arm_with_self_filter_collision.urdf (robot description, URDF)
Before this commit: robot Arm_collision_only, 9 links, 8 joints
Links:
- link link2: geometry collision box size=0.086 0.138 0.155; collision cylinder length=0.155 radius=0.071

Commit message: Refine self-filter collision geometry

File: src/arm_description/urdf/Arm_with_self_filter_collision.urdf (robot description, URDF)
Before this commit: robot Arm_collision_only, 9 links, 8 joints
Links:
- link link4: geometry collision box size=0.090 0.170 0.070; collision cylinder length=0.070 radius=0.03
- link wrist_link1: geometry collision box size=0.090 0.015 0.060; collision cylinder length=0.030 radius=0.020

Commit message: Refine self-filter geometry after RViz audit

File: src/arm_description/urdf/Arm_with_self_filter_collision.urdf (robot description, URDF)
Before this commit: robot Arm_collision_only, 9 links, 8 joints
Links:
- link wrist_link3: geometry collision box size=0.015 0.015 0.055; collision box size=0.035 0.025 0.055

Commit message: Refine wrist_link1 self-filter geometry

File: src/arm_description/urdf/Arm_with_self_filter_collision.urdf (robot description, URDF)
Before this commit: robot Arm_collision_only, 9 links, 8 joints
Links:
- link wrist_link1: geometry collision box size=0.040 0.030 0.030; collision box size=0.090 0.015 0.060

Commit message: Refine self-filter geometry after multi-link RViz audit

File: src/arm_description/urdf/Arm_with_self_filter_collision.urdf (robot description, URDF)
Before this commit: robot Arm_collision_only, 9 links, 8 joints
Links:
- link link1: geometry collision box size=0.115 0.115 0.125; collision cylinder length=0.025 radius=0.073
- link link3: geometry collision box size=0.025 0.056 0.055; collision box size=0.090 0.102 0.132
- link wrist_link2: geometry collision cylinder length=0.065 radius=0.038; visual mesh filename=package://arm_description/meshes/wrist_link2.STL
- link wrist_link3: geometry collision box size=0.015 0.015 0.055; collision box size=0.035 0.025 0.055

Commit message: Refine remaining self-filter geometry

File: src/arm_description/urdf/Arm_with_self_filter_collision.urdf (robot description, URDF)
Before this commit: robot Arm_collision_only, 9 links, 8 joints
Links:
- link link3: geometry collision box size=0.025 0.056 0.055; collision box size=0.090 0.102 0.132
- link link4: geometry collision box size=0.090 0.170 0.070; collision cylinder length=0.070 radius=0.03
- link wrist_link3: geometry collision box size=0.015 0.015 0.055; collision box size=0.035 0.025 0.055

Commit message: Polish residual self-filter geometry

File: src/arm_description/urdf/Arm_with_self_filter_collision.urdf (robot description, URDF)
Before this commit: robot Arm_collision_only, 9 links, 8 joints
Links:
- link link1: geometry collision box size=0.118 0.115 0.125; collision cylinder length=0.025 radius=0.073
- link link2: geometry collision box size=0.086 0.138 0.155; collision cylinder length=0.02 radius=0.045
- link link3: geometry collision box size=0.025 0.058 0.058; collision box size=0.090 0.102 0.132
- link link4: geometry collision box size=0.090 0.180 0.070; collision cylinder length=0.070 radius=0.03
- link wrist_link3: geometry collision box size=0.015 0.015 0.055; collision box size=0.035 0.025 0.055

Commit message: Finish residual self-filter geometry refinement

File: src/arm_description/urdf/Arm_with_self_filter_collision.urdf (robot description, URDF)
Before this commit: robot Arm_collision_only, 9 links, 8 joints
Links:
- link link1: geometry collision box size=0.118 0.115 0.125; collision cylinder length=0.025 radius=0.075
- link link4: geometry collision box size=0.090 0.180 0.075; collision cylinder length=0.070 radius=0.03
- link wrist_link3: geometry collision box size=0.016 0.016 0.055; collision box size=0.037 0.027 0.057

Commit message: Update base self-filter geometry

File: src/arm_description/urdf/Arm_with_self_filter_collision.urdf (robot description, URDF)
Before this commit: robot Arm_collision_only, 9 links, 8 joints
Links:
- link base_link: geometry collision cylinder length=0.0160 radius=0.095; collision cylinder length=0.068 radius=0.078
- link link1: geometry collision box size=0.118 0.115 0.125; collision cylinder length=0.035 radius=0.075

Commit message: Certify complete self-filter visual coverage

File: src/arm_description/urdf/Arm_with_self_filter_collision.urdf (robot description, URDF)
Before this commit: robot Arm_collision_only, 9 links, 8 joints
Links:
- link base_link: geometry collision cylinder length=0.0155 radius=0.095; collision cylinder length=0.068 radius=0.078
